Commit message: Embed current P2 control parameters in URDF assets

File: protomotions/data/assets/astro_p2/urdf/astro_p2_30dof_mesh_collision.urdf (robot description, URDF)
Before this commit: robot astro, 37 links, 36 joints
Joints:
- joint head_joint: limit lower=-0.61 upper=0.61 effort=10 velocity=20.94 -> lower=-0.61 upper=0.61 effort=10.0 velocity=20.94
- joint left_ankle_pitch_joint: limit lower=-0.79 upper=0.52 effort=60 velocity=26.18 -> lower=-0.79 upper=0.52 effort=60.0 velocity=26.18
- joint left_ankle_roll_joint: limit lower=-0.35 upper=0.35 effort=45 velocity=26.18 -> lower=-0.35 upper=0.35 effort=45.0 velocity=26.18
- joint left_elbow_joint: limit lower=-0.52 upper=1.66 effort=30 velocity=26.18 -> lower=-0.52 upper=1.66 effort=30.0 velocity=26.18
- joint left_hip_pitch_joint: limit lower=-2.62 upper=2.62 effort=130 velocity=23.04 -> lower=-2.62 upper=2.62 effort=130.0 velocity=23.04
- joint left_hip_roll_joint: limit lower=-0.26 upper=2.79 effort=130 velocity=23.04 -> lower=-0.26 upper=2.79 effort=130.0 velocity=23.04
- joint left_hip_yaw_joint: limit lower=-1.57 upper=3.67 effort=130 velocity=23.04 -> lower=-1.57 upper=3.67 effort=130.0 velocity=23.04
- joint left_knee_joint: limit lower=-0.09 upper=2.44 effort=130 velocity=23.04 -> lower=-0.09 upper=2.44 effort=130.0 velocity=23.04
- joint left_shoulder_pitch_joint: limit lower=-2.79 upper=2.79 effort=30 velocity=26.18 -> lower=-2.79 upper=2.79 effort=30.0 velocity=26.18
- joint left_shoulder_roll_joint: limit lower=-0.26 upper=2.62 effort=30 velocity=26.18 -> lower=-0.26 upper=2.62 effort=30.0 velocity=26.18
- joint left_shoulder_yaw_joint: limit lower=-1.92 upper=1.92 effort=30 velocity=26.18 -> lower=-1.92 upper=1.92 effort=30.0 velocity=26.18
- joint left_wrist_pitch_joint: limit lower=-1.31 upper=1.31 effort=10 velocity=20.94 -> lower=-1.31 upper=1.31 effort=10.0 velocity=20.94
- joint left_wrist_roll_joint: limit lower=-1.92 upper=1.92 effort=30 velocity=26.18 -> lower=-1.92 upper=1.92 effort=30.0 velocity=26.18
- joint left_wrist_yaw_joint: limit lower=-1.31 upper=1.31 effort=10 velocity=20.94 -> lower=-1.31 upper=1.31 effort=10.0 velocity=20.94
- joint right_ankle_pitch_joint: limit lower=-0.79 upper=0.52 effort=60 velocity=26.18 -> lower=-0.79 upper=0.52 effort=60.0 velocity=26.18
- joint right_ankle_roll_joint: limit lower=-0.35 upper=0.35 effort=45 velocity=26.18 -> lower=-0.35 upper=0.35 effort=45.0 velocity=26.18
- joint right_elbow_joint: limit lower=-0.52 upper=1.66 effort=30 velocity=26.18 -> lower=-0.52 upper=1.66 effort=30.0 velocity=26.18
- joint right_hip_pitch_joint: limit lower=-2.62 upper=2.62 effort=130 velocity=23.04 -> lower=-2.62 upper=2.62 effort=130.0 velocity=23.04
- joint right_hip_roll_joint: limit lower=-2.79 upper=0.26 effort=130 velocity=23.04 -> lower=-2.79 upper=0.26 effort=130.0 velocity=23.04
- joint right_hip_yaw_joint: limit lower=-3.67 upper=1.57 effort=130 velocity=23.04 -> lower=-3.67 upper=1.57 effort=130.0 velocity=23.04
- joint right_knee_joint: limit lower=-0.09 upper=2.44 effort=130 velocity=23.04 -> lower=-0.09 upper=2.44 effort=130.0 velocity=23.04
- joint right_shoulder_pitch_joint: limit lower=-2.79 upper=2.79 effort=30 velocity=26.18 -> lower=-2.79 upper=2.79 effort=30.0 velocity=26.18
- joint right_shoulder_roll_joint: limit lower=-2.62 upper=0.26 effort=30 velocity=26.18 -> lower=-2.62 upper=0.26 effort=30.0 velocity=26.18
- joint right_shoulder_yaw_joint: limit lower=-1.92 upper=1.92 effort=30 velocity=26.18 -> lower=-1.92 upper=1.92 effort=30.0 velocity=26.18
- joint right_wrist_pitch_joint: limit lower=-1.31 upper=1.31 effort=10 velocity=20.94 -> lower=-1.31 upper=1.31 effort=10.0 velocity=20.94
- joint right_wrist_roll_joint: limit lower=-1.92 upper=1.92 effort=30 velocity=26.18 -> lower=-1.92 upper=1.92 effort=30.0 velocity=26.18
- joint right_wrist_yaw_joint: limit lower=-1.31 upper=1.31 effort=10 velocity=20.94 -> lower=-1.31 upper=1.31 effort=10.0 velocity=20.94
- joint waist_pitch_joint: limit lower=-0.37 upper=0.44 effort=60 velocity=26.18 -> lower=-0.37 upper=0.44 effort=60.0 velocity=26.18
- joint waist_roll_joint: limit lower=-0.28 upper=0.28 effort=50 velocity=26.18 -> lower=-0.28 upper=0.28 effort=50.0 velocity=26.18
- joint waist_yaw_joint: limit lower=-1.57 upper=3.67 effort=130 velocity=13.04 -> lower=-1.57 upper=3.67 effort=130.0 velocity=13.04

File: protomotions/data/assets/astro_p2/urdf/astro_p2_30dof_primitive_collision.urdf (robot description, URDF)
Before this commit: robot astro, 37 links, 36 joints
Joints:
- joint head_joint: limit lower=-0.61 upper=0.61 effort=10 velocity=20.94 -> lower=-0.61 upper=0.61 effort=10.0 velocity=20.94
- joint left_ankle_pitch_joint: limit lower=-0.79 upper=0.52 effort=60 velocity=26.18 -> lower=-0.79 upper=0.52 effort=60.0 velocity=26.18
- joint left_ankle_roll_joint: limit lower=-0.35 upper=0.35 effort=45 velocity=26.18 -> lower=-0.35 upper=0.35 effort=45.0 velocity=26.18
- joint left_elbow_joint: limit lower=-0.52 upper=1.66 effort=30 velocity=26.18 -> lower=-0.52 upper=1.66 effort=30.0 velocity=26.18
- joint left_hip_pitch_joint: limit lower=-2.62 upper=2.62 effort=130 velocity=23.04 -> lower=-2.62 upper=2.62 effort=130.0 velocity=23.04
- joint left_hip_roll_joint: limit lower=-0.26 upper=2.79 effort=130 velocity=23.04 -> lower=-0.26 upper=2.79 effort=130.0 velocity=23.04
- joint left_hip_yaw_joint: limit lower=-1.57 upper=3.67 effort=130 velocity=23.04 -> lower=-1.57 upper=3.67 effort=130.0 velocity=23.04
- joint left_knee_joint: limit lower=-0.09 upper=2.44 effort=130 velocity=23.04 -> lower=-0.09 upper=2.44 effort=130.0 velocity=23.04
- joint left_shoulder_pitch_joint: limit lower=-2.79 upper=2.79 effort=30 velocity=26.18 -> lower=-2.79 upper=2.79 effort=30.0 velocity=26.18
- joint left_shoulder_roll_joint: limit lower=-0.26 upper=2.62 effort=30 velocity=26.18 -> lower=-0.26 upper=2.62 effort=30.0 velocity=26.18
- joint left_shoulder_yaw_joint: limit lower=-1.92 upper=1.92 effort=30 velocity=26.18 -> lower=-1.92 upper=1.92 effort=30.0 velocity=26.18
- joint left_wrist_pitch_joint: limit lower=-1.31 upper=1.31 effort=10 velocity=20.94 -> lower=-1.31 upper=1.31 effort=10.0 velocity=20.94
- joint left_wrist_roll_joint: limit lower=-1.92 upper=1.92 effort=30 velocity=26.18 -> lower=-1.92 upper=1.92 effort=30.0 velocity=26.18
- joint left_wrist_yaw_joint: limit lower=-1.31 upper=1.31 effort=10 velocity=20.94 -> lower=-1.31 upper=1.31 effort=10.0 velocity=20.94
- joint right_ankle_pitch_joint: limit lower=-0.79 upper=0.52 effort=60 velocity=26.18 -> lower=-0.79 upper=0.52 effort=60.0 velocity=26.18
- joint right_ankle_roll_joint: limit lower=-0.35 upper=0.35 effort=45 velocity=26.18 -> lower=-0.35 upper=0.35 effort=45.0 velocity=26.18
- joint right_elbow_joint: limit lower=-0.52 upper=1.66 effort=30 velocity=26.18 -> lower=-0.52 upper=1.66 effort=30.0 velocity=26.18
- joint right_hip_pitch_joint: limit lower=-2.62 upper=2.62 effort=130 velocity=23.04 -> lower=-2.62 upper=2.62 effort=130.0 velocity=23.04
- joint right_hip_roll_joint: limit lower=-2.79 upper=0.26 effort=130 velocity=23.04 -> lower=-2.79 upper=0.26 effort=130.0 velocity=23.04
- joint right_hip_yaw_joint: limit lower=-3.67 upper=1.57 effort=130 velocity=23.04 -> lower=-3.67 upper=1.57 effort=130.0 velocity=23.04
- joint right_knee_joint: limit lower=-0.09 upper=2.44 effort=130 velocity=23.04 -> lower=-0.09 upper=2.44 effort=130.0 velocity=23.04
- joint right_shoulder_pitch_joint: limit lower=-2.79 upper=2.79 effort=30 velocity=26.18 -> lower=-2.79 upper=2.79 effort=30.0 velocity=26.18
- joint right_shoulder_roll_joint: limit lower=-2.62 upper=0.26 effort=30 velocity=26.18 -> lower=-2.62 upper=0.26 effort=30.0 velocity=26.18
- joint right_shoulder_yaw_joint: limit lower=-1.92 upper=1.92 effort=30 velocity=26.18 -> lower=-1.92 upper=1.92 effort=30.0 velocity=26.18
- joint right_wrist_pitch_joint: limit lower=-1.31 upper=1.31 effort=10 velocity=20.94 -> lower=-1.31 upper=1.31 effort=10.0 velocity=20.94
- joint right_wrist_roll_joint: limit lower=-1.92 upper=1.92 effort=30 velocity=26.18 -> lower=-1.92 upper=1.92 effort=30.0 velocity=26.18
- joint right_wrist_yaw_joint: limit lower=-1.31 upper=1.31 effort=10 velocity=20.94 -> lower=-1.31 upper=1.31 effort=10.0 velocity=20.94
- joint waist_pitch_joint: limit lower=-0.37 upper=0.44 effort=60 velocity=26.18 -> lower=-0.37 upper=0.44 effort=60.0 velocity=26.18
- joint waist_roll_joint: limit lower=-0.28 upper=0.28 effort=50 velocity=26.18 -> lower=-0.28 upper=0.28 effort=50.0 velocity=26.18
- joint waist_yaw_joint: limit lower=-1.57 upper=3.67 effort=130 velocity=13.04 -> lower=-1.57 upper=3.67 effort=130.0 velocity=13.04

File: protomotions/data/assets/astro_p2/urdf/astro_p2_retarget.urdf (robot description, URDF)
Before this commit: robot astro, 39 links, 38 joints
Joints:
- joint head_joint: limit lower=-0.61 upper=0.61 effort=10 velocity=20.94 -> lower=-0.61 upper=0.61 effort=10.0 velocity=20.94
- joint left_ankle_pitch_joint: limit lower=-0.79 upper=0.52 effort=60 velocity=26.18 -> lower=-0.79 upper=0.52 effort=60.0 velocity=26.18
- joint left_ankle_roll_joint: limit lower=-0.35 upper=0.35 effort=45 velocity=26.18 -> lower=-0.35 upper=0.35 effort=45.0 velocity=26.18
- joint left_elbow_joint: limit lower=-0.52 upper=1.66 effort=30 velocity=26.18 -> lower=-0.52 upper=1.66 effort=30.0 velocity=26.18
- joint left_hip_pitch_joint: limit lower=-2.62 upper=2.62 effort=130 velocity=23.04 -> lower=-2.62 upper=2.62 effort=130.0 velocity=23.04
- joint left_hip_roll_joint: limit lower=-0.26 upper=2.79 effort=130 velocity=23.04 -> lower=-0.26 upper=2.79 effort=130.0 velocity=23.04
- joint left_hip_yaw_joint: limit lower=-1.57 upper=3.67 effort=130 velocity=23.04 -> lower=-1.57 upper=3.67 effort=130.0 velocity=23.04
- joint left_knee_joint: limit lower=-0.09 upper=2.44 effort=130 velocity=23.04 -> lower=-0.09 upper=2.44 effort=130.0 velocity=23.04
- joint left_shoulder_pitch_joint: limit lower=-2.79 upper=2.79 effort=30 velocity=26.18 -> lower=-2.79 upper=2.79 effort=30.0 velocity=26.18
- joint left_shoulder_roll_joint: limit lower=-0.26 upper=2.62 effort=30 velocity=26.18 -> lower=-0.26 upper=2.62 effort=30.0 velocity=26.18
- joint left_shoulder_yaw_joint: limit lower=-1.92 upper=1.92 effort=30 velocity=26.18 -> lower=-1.92 upper=1.92 effort=30.0 velocity=26.18
- joint left_wrist_pitch_joint: limit lower=-1.31 upper=1.31 effort=10 velocity=20.94 -> lower=-1.31 upper=1.31 effort=10.0 velocity=20.94
- joint left_wrist_roll_joint: limit lower=-1.92 upper=1.92 effort=30 velocity=26.18 -> lower=-1.92 upper=1.92 effort=30.0 velocity=26.18
- joint left_wrist_yaw_joint: limit lower=-1.31 upper=1.31 effort=10 velocity=20.94 -> lower=-1.31 upper=1.31 effort=10.0 velocity=20.94
- joint right_ankle_pitch_joint: limit lower=-0.79 upper=0.52 effort=60 velocity=26.18 -> lower=-0.79 upper=0.52 effort=60.0 velocity=26.18
- joint right_ankle_roll_joint: limit lower=-0.35 upper=0.35 effort=45 velocity=26.18 -> lower=-0.35 upper=0.35 effort=45.0 velocity=26.18
- joint right_elbow_joint: limit lower=-0.52 upper=1.66 effort=30 velocity=26.18 -> lower=-0.52 upper=1.66 effort=30.0 velocity=26.18
- joint right_hip_pitch_joint: limit lower=-2.62 upper=2.62 effort=130 velocity=23.04 -> lower=-2.62 upper=2.62 effort=130.0 velocity=23.04
- joint right_hip_roll_joint: limit lower=-2.79 upper=0.26 effort=130 velocity=23.04 -> lower=-2.79 upper=0.26 effort=130.0 velocity=23.04
- joint right_hip_yaw_joint: limit lower=-3.67 upper=1.57 effort=130 velocity=23.04 -> lower=-3.67 upper=1.57 effort=130.0 velocity=23.04
- joint right_knee_joint: limit lower=-0.09 upper=2.44 effort=130 velocity=23.04 -> lower=-0.09 upper=2.44 effort=130.0 velocity=23.04
- joint right_shoulder_pitch_joint: limit lower=-2.79 upper=2.79 effort=30 velocity=26.18 -> lower=-2.79 upper=2.79 effort=30.0 velocity=26.18
- joint right_shoulder_roll_joint: limit lower=-2.62 upper=0.26 effort=30 velocity=26.18 -> lower=-2.62 upper=0.26 effort=30.0 velocity=26.18
- joint right_shoulder_yaw_joint: limit lower=-1.92 upper=1.92 effort=30 velocity=26.18 -> lower=-1.92 upper=1.92 effort=30.0 velocity=26.18
- joint right_wrist_pitch_joint: limit lower=-1.31 upper=1.31 effort=10 velocity=20.94 -> lower=-1.31 upper=1.31 effort=10.0 velocity=20.94
- joint right_wrist_roll_joint: limit lower=-1.92 upper=1.92 effort=30 velocity=26.18 -> lower=-1.92 upper=1.92 effort=30.0 velocity=26.18
- joint right_wrist_yaw_joint: limit lower=-1.31 upper=1.31 effort=10 velocity=20.94 -> lower=-1.31 upper=1.31 effort=10.0 velocity=20.94
- joint waist_pitch_joint: limit lower=-0.37 upper=0.44 effort=60 velocity=26.18 -> lower=-0.37 upper=0.44 effort=60.0 velocity=26.18
- joint waist_roll_joint: limit lower=-0.28 upper=0.28 effort=50 velocity=26.18 -> lower=-0.28 upper=0.28 effort=50.0 velocity=26.18
- joint waist_yaw_joint: limit lower=-1.57 upper=3.67 effort=130 velocity=13.04 -> lower=-1.57 upper=3.67 effort=130.0 velocity=13.04
